Commit message: fixes

File: pantilt_description/urdf/pantilt.urdf.xacro (robot description, xacro)
@@ -4,7 +4,7 @@
     <xacro:arg name="is_sim" default="true"/>
     <!-- Include Gazebo Parameters -->
-    <xacro:include filename="$(find pantilt_description)/urdf/pantilt_gazebo.xacro" />
+    <!-- <xacro:include filename="$(find pantilt_description)/urdf/pantilt_gazebo.xacro" /> -->
     <!-- Include ros2_control Plugins -->
-    <xacro:include filename="$(find pantilt_description)/urdf/pantilt_ros2_control.xacro" />
+    <!-- <xacro:include filename="$(find pantilt_description)/urdf/pantilt_ros2_control.xacro" /> -->
      <!-- Include camera -->
     <xacro:include filename="$(find pantilt_description)/urdf/pantilt_camera.xacro" />

File: pantilt_description/urdf/pantilt_camera.xacro (robot description, xacro)
@@ -9,15 +9,15 @@
         <visual>
             <geometry>
-                <box size=".01 .04 .04"/>
+                <box size="0.01 0.04 0.04"/>
             </geometry>
             <material name="white"/>
         </visual>
-<!--         <collision>
+        <collision>
            <geometry>
-                <box size="0.010 0.03 0.03"/>
+                <box size="0.01 0.04 0.04"/>
             </geometry>
-        </collision> -->
+        </collision>
         <visual>
-            <origin xyz="0 0 0 .025"/>
+            <origin xyz="0 0 0.025"/>
             <geometry>
                 <cylinder radius="0.002" length="0.01"/>
@@ -25,10 +25,10 @@
             <material name="white"/>
         </visual>
-<!--          <collision>
-            <origin xyz="0 0 -0.05"/>
+        <collision>
+            <origin xyz="0 0 0.025"/>
            <geometry>
-                 <cylinder radius="0.002" length="0.1"/>
+                 <cylinder radius="0.002" length="0.01"/>
             </geometry>
-        </collision>  -->
+        </collision>
     </link>
     <joint name="camera_optical_joint" type="fixed">
